File: kicad/pro_mini.kicad_pcb (KiCad board)
At the start: 2 copper layers, 17.8 x 33 mm, 11 parts, among them IC1 ATMEGA328P-A, P1 FTDI, P2 DIGITAL, P3 CONN_01X12

Commit message: Layout
Parts:
- added C5: 1uF, Capacitors_SMD:C_0805_HandSoldering, F.Cu at (105.3, 105.0)
- added C6: 1uF, Capacitors_SMD:C_0805_HandSoldering, F.Cu at (112.0, 105.0)
- added U1: MCP1700T-3302E, TO_SOT_Packages_SMD:SOT89-3_Housing_Handsoldering, F.Cu at (108.7, 106.6)
- moved R2 38.8 mm to (106.5, 130.9)
- moved C1 36.9 mm to (105.4, 112.0), turned to 90 degrees
- moved C2 35.2 mm to (114.5, 131.0), turned to 180 degrees
- moved C4 28.3 mm to (113.9, 105.0), turned to 90 degrees
- moved C3 6.80 mm to (114.9, 109.8), turned to 90 degrees
- moved R1 5.14 mm to (113.0, 109.8), turned to 270 degrees
- moved D1 5.08 mm to (110.6, 129.2), turned to 180 degrees
Connections:
- P2 pad 11: A5 -> A4
- P2 pad 12: A4 -> A5
- P3 pad 12: Net-(P3-Pad12) -> RAW
Routing:
- net GND: track 0.00 -> 82.3 mm, vias 0 -> 4
- net VCC: track 0.00 -> 52.9 mm, vias 0 -> 1
- net RAW: track 0.00 -> 24.2 mm
- net A6: track 0.00 -> 21.2 mm, vias 0 -> 1
- net A5: track 0.00 -> 21.1 mm, vias 0 -> 1
- net A7: track 0.00 -> 20.6 mm, vias 0 -> 1
- net SCK: track 0.00 -> 20.2 mm, vias 0 -> 2
- net A4: track 0.00 -> 20.2 mm, vias 0 -> 1
- net RXI: track 0.00 -> 18.9 mm, vias 0 -> 1
- net TXO: track 0.00 -> 16.8 mm, vias 0 -> 1
- net D10: track 0.00 -> 14.6 mm
- net MOSI: track 0.00 -> 12.3 mm
- net /AREF: track 0.00 -> 11.4 mm, vias 0 -> 2
- net D2: track 0.00 -> 9.89 mm, vias 0 -> 1
- net MISO: track 0.00 -> 9.69 mm
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- added copper zone on B.Cu, net GND
- added copper zone on F.Cu, net GND
Other:
- net class RAW added: clearance 0.3048, trace_width 0.3048, via_dia 0.6858, via_drill 0.3556
- net class VCC added: clearance 0.3048, trace_width 0.3048, via_dia 0.6858, via_drill 0.3556

Commit message: Room for pin labels
Parts:
- moved C5 3.90 mm to (108.9, 103.5), turned to 180 degrees
- moved U1 2.06 mm to (109.3, 108.5)
- moved C1 0.81 mm to (106.2, 112.0)
- moved C4 0.73 mm to (114.6, 104.7)
- moved C6 0.64 mm to (112.5, 104.7)
- moved C3 0.28 mm to (114.6, 109.7)
- moved R1 0.27 mm to (112.8, 109.7)
Routing:
- net GND: track 82.3 -> 90.0 mm, vias 4 -> 3
- net RAW: track 24.2 -> 18.8 mm
- net VCC: track 52.9 -> 48.2 mm
- net DTR: track 9.10 -> 9.79 mm
- net A7: track 20.6 -> 21.3 mm
Other:
- board text added: "A6"
- board text added: "A7"

Commit message: Pin labels
Parts:
- moved R2 1.20 mm to (107.7, 131.0)
- moved C2 0.98 mm to (113.5, 131.1)
- moved D1 0.08 mm to (110.5, 129.2)
Routing:
- net GND: track 90.0 -> 98.9 mm, vias 3 -> 6
- net Net-(D1-Pad2): track 2.87 -> 2.14 mm
Other:
- board text added: "A0"
- board text added: "A1"
- board text added: "A2"
- board text added: "A3"
- board text added: "A4"
- board text added: "A5"
- board text added: "D10"
- board text added: "D11"
- board text added: "D12"
- board text added: "D13"
- board text added: "D2"
- board text added: "D3"
- board text added: "D4"
- board text added: "D5"
- board text added: "D6"
- board text added: "D7"
- board text added: "D8"
- board text added: "D9"
- board text added: "DTR"
- board text added: "GND"
- board text added: "RAW"
- board text added: "RXI"
- board text added: "TXO"
- board text added: "VCC"

Commit message: Theapi tiny logo
Parts:
- added REF**: TheApiLogoTiny, theapi_graphics:TheApiLogoTiny, F.Cu at (106.2, 105.8)
Changed lines of the file:
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@@
 (kicad_pcb (version 4) (host pcbnew 4.0.1-stable)
   (general
-    (links 54)
+    (links 0)
     (no_connects 0)
     (area 101.524999 98.984999 119.455001 132.155001)
@@
     (tracks 280)
     (zones 0)
-    (modules 14)
+    (modules 15)
     (nets 32)
   )
@@
     (pad_to_mask_clearance 0.2)
     (aux_axis_origin 0 0)
-    (visible_elements FFFFF77F)
+    (visible_elements 7FFFFFFF)
     (pcbplotparams
       (layerselection 0x00030_80000001)
@@
     )
   )
+  (module theapi_graphics:TheApiLogoTiny (layer F.Cu)
+    (at 106.172 105.791)
+    (fp_text reference REF** (at 0 0.5) (layer F.SilkS) hide
+      (effects (font (size 1 1) (thickness 0.15)))
+    )
+    (fp_text value TheApiLogoTiny (at 0 -0.5) (layer F.Fab) hide
+      (effects (font (size 1 1) (thickness 0.15)))
+    )
+    (fp_line (start 0.26 4.07) (end 0.42 3.55) (layer F.Mask) (width 0.1016))
+    (fp_line (start 0.3 3.85) (end 0.26 4.07) (layer F.Mask) (width 0.1016))
+    (fp_line (start 0.18 3.57) (end 0.3 3.85) (layer F.Mask) (width 0.1016))
+    (fp_line (start -0.04 3.27) (end 0.18 3.57) (layer F.Mask) (width 0.1016))
+    (fp_line (start -0.13 2.84) (end -0.04 3.27) (layer F.Mask) (width 0.1016))
+    (fp_line (start 0.24 2.85) (end 0.24 2.68) (layer F.Mask) (width 0.1016))
+    (fp_line (start 0.26 2.95) (end 0.24 2.85) (layer F.Mask) (width 0.1016))
+    (fp_line (start 0.21 3.04) (end 0.26 2.95) (layer F.Mask) (width 0.1016))
+    (fp_line (start 0.09 3.07) (end 0.21 3.04) (layer F.Mask) (width 0.1016))
+    (fp_line (start -0.03 2.94) (end 0.09 3.07) (layer F.Mask) (width 0.1016))
+    (fp_line (start -0.1 2.75) (end -0.03 2.94) (layer F.Mask) (width 0.1016))
+    (fp_line (start 0.42 2.75) (end 0.33 2.62) (layer F.Mask) (width 0.1016))
+    (fp_line (start 0.55 2.78) (end 0.42 2.75) (layer F.Mask) (width 0.1016))
+    (fp_line (start 0.66 2.74) (end 0.55 2.78) (layer F.Mask) (width 0.1016))
+    (fp_line (start 0.7 2.64) (end 0.66 2.74) (layer F.Mask) (width 0.1016))
+    (fp_line (start 0.7 2.5) (end 0.7 2.64) (layer F.Mask) (width 0.1016))
+    (fp_line (start 0.6 2.36) (end 0.7 2.5) (layer F.Mask) (width 0.1016))
+    (fp_line (start 0.42 2.25) (end 0.6 2.36) (layer F.Mask) (width 0.1016))
+    (fp_line (start 0.52 2.22) (end 0.42 2.22) (layer F.Mask) (width 0.1016))
+    (fp_line (start 0.67 2.21) (end 0.52 2.22) (layer F.Mask) (width 0.1016))
+    (fp_line (start 0.77 2.14) (end 0.67 2.21) (layer F.Mask) (width 0.1016))
+    (fp_line (start 0.75 1.99) (end 0.77 2.14) (layer F.Mask) (width 0.1016))
+    (fp_line (start 0.64 1.89) (end 0.75 1.99) (layer F.Mask) (width 0.1016))
+    (fp_line (start 0.27 1.9) (end 0.64 1.89) (layer F.Mask) (width 0.1016))
+    (fp_line (start 0.39 1.77) (end 0.3 1.91) (layer F.Mask) (width 0.1016))
+    (fp_line (start 0.41 1.66) (end 0.39 1.77) (layer F.Mask) (width 0.1016))
+    (fp_line (start 0.36 1.55) (end 0.41 1.66) (layer F.Mask) (width 0.1016))
+    (fp_line (start 0.19 1.52) (end 0.36 1.55) (layer F.Mask) (width 0.1016))
+    (fp_line (start 0.03 1.58) (end 0.19 1.52) (layer F.Mask) (width 0.1016))
+    (fp_line (start -0.06 1.85) (end 0.03 1.58) (layer F.Mask) (width 0.1016))
+    (fp_line (start -0.16 2.76) (end -0.17 2.73) (layer F.Mask) (width 0.1016))
+    (fp_line (start -0.13 2.74) (end -0.16 2.76) (layer F.Mask) (width 0.1016))
+    (fp_line (start -0.15 2.76) (end -0.13 2.74) (layer F.Mask) (width 0.1016))
+    (fp_line (start -0.17 2.87) (end -0.15 2.76) (layer F.Mask) (width 0.1016))
+    (fp_line (start -0.23 2.98) (end -0.17 2.87) (layer F.Mask) (width 0.1016))
+    (fp_line (start -0.35 3.02) (end -0.23 2.98) (layer F.Mask) (width 0.1016))
+    (fp_line (start -0.46 2.98) (end -0.35 3.02) (layer F.Mask) (width 0.1016))
+    (fp_line (start -0.47 2.79) (end -0.46 2.98) (layer F.Mask) (width 0.1016))
+    (fp_line (start -0.39 2.59) (end -0.47 2.79) (layer F.Mask) (width 0.1016))
+    (fp_line (start -0.66 2.63) (end -0.41 2.57) (layer F.Mask) (width 0.1016))
+    (fp_line (start -0.78 2.55) (end -0.66 2.63) (layer F.Mask) (width 0.1016))
+    (fp_line (start -0.82 2.42) (end -0.78 2.55) (layer F.Mask) (width 0.1016))
+    (fp_line (start -0.73 2.27) (end -0.82 2.42) (layer F.Mask) (width 0.1016))
+    (fp_line (start -0.46 2.22) (end -0.73 2.27) (layer F.Mask) (width 0.1016))
+    (fp_line (start -0.68 2.1) (end -0.47 2.15) (layer F.Mask) (width 0.1016))
+    (fp_line (start -0.79 1.93) (end -0.68 2.1) (layer F.Mask) (width 0.1016))
+    (fp_line (start -0.68 1.74) (end -0.79 1.93) (layer F.Mask) (width 0.1016))
+    (fp_line (start -0.4 1.67) (end -0.68 1.74) (layer F.Mask) (width 0.1016))
+    (fp_line (start -0.13 1.81) (end -0.4 1.67) (layer F.Mask) (width 0.1016))
+    (fp_line (start 0.04 2.48) (end 0.16 2.39) (layer F.Mask) (width 0.0762))
+    (fp_line (start -0.09 2.49) (end 0.04 2.48) (layer F.Mask) (width 0.0762))
+    (fp_line (start -0.21 2.42) (end -0.09 2.49) (layer F.Mask) (width 0.0762))
+    (fp_circle (center -0.16 2.2) (end -0.13 2.21) (layer F.Mask) (width 0.15))
+    (fp_circle (center -0.02 2.28) (end 0.39 2.28) (layer F.Mask) (width 0.127))
+    (fp_circle (center 0.12 2.2) (end 0.15 2.21) (layer F.Mask) (width 0.15))
+  )
   (gr_text VCC (at 116.332 110.49 90) (layer F.SilkS)
